Commit message: inclu landpad

File: magni_description/urdf/magni.urdf.xacro (robot description, xacro)
@@ -1,14 +1,14 @@
 <?xml version="1.0"?>
 <robot xmlns:xacro="http://wiki.ros.org/xacro" name="magni">
-  <xacro:arg name="sonars_installed" default="true"/>
-  <xacro:property name="sonars_installed" value="$(arg sonars_installed)"/>
-  <xacro:arg name="shell_installed" default="false"/>
-  <xacro:property name="shell_installed" value="$(arg shell_installed)"/>
-  <xacro:arg name="tower_installed" default="false"/>
-  <xacro:property name="tower_installed" value="$(arg tower_installed)"/>
-  <xacro:arg name="camera_extrinsics_file" default=""/>
-  <xacro:property name="camera_extrinsics_file" value="$(arg camera_extrinsics_file)"/>
-  <xacro:arg name="lidar_extrinsics_file" default=""/>
-  <xacro:property name="lidar_extrinsics_file" value="$(arg lidar_extrinsics_file)"/>
+  <xacro:arg name="sonars_installed" default="true" />
+  <xacro:property name="sonars_installed" value="$(arg sonars_installed)" />
+  <xacro:arg name="shell_installed" default="false" />
+  <xacro:property name="shell_installed" value="$(arg shell_installed)" />
+  <xacro:arg name="tower_installed" default="false" />
+  <xacro:property name="tower_installed" value="$(arg tower_installed)" />
+  <xacro:arg name="camera_extrinsics_file" default="" />
+  <xacro:property name="camera_extrinsics_file" value="$(arg camera_extrinsics_file)" />
+  <xacro:arg name="lidar_extrinsics_file" default="" />
+  <xacro:property name="lidar_extrinsics_file" value="$(arg lidar_extrinsics_file)" />
   <xacro:property name="wheel_r" value="0.1" />
   <xacro:property name="wheel_xpos" value="0.11" />
@@ -19,4 +19,5 @@
   <xacro:include filename="$(find magni_description)/urdf/sensors/raspi_camera.xacro" />
   <xacro:include filename="$(find magni_description)/urdf/sensors/ur50_lidar.xacro" />
+  <xacro:include filename="$(find magni_description)/urdf/sensors/teste.xacro" />
   <!-- Robot base_link -->
   <link name="base_link">
@@ -27,5 +28,5 @@
       </geometry>
     </visual>
-	<visual>
+    <visual>
       <origin xyz="${-wheel_xpos-0.169} 0.17 ${-wheel_r+0.09}" rpy="0 0 ${pi}" />
       <geometry>
@@ -33,5 +34,5 @@
       </geometry>
     </visual>
-	<visual>
+    <visual>
       <origin xyz="${-wheel_xpos-0.169} -0.17 ${-wheel_r+0.09}" rpy="0 0 ${pi}" />
       <geometry>
@@ -40,7 +41,7 @@
     </visual>
     <collision>
-	  <origin xyz="${-wheel_xpos} 0 ${-wheel_r+0.151}" rpy="0 0 0" />
-      <geometry>
-        <box size="0.398 0.268 0.160"/>
+      <origin xyz="${-wheel_xpos} 0 ${-wheel_r+0.151}" rpy="0 0 0" />
+      <geometry>
+        <box size="0.398 0.268 0.160" />
       </geometry>
     </collision>
@@ -48,5 +49,5 @@
       <origin xyz="${-wheel_xpos-0.026} 0 ${-wheel_r+0.248}" rpy="0 0 0" />
       <geometry>
-        <box size="0.375 0.268 0.034"/>
+        <box size="0.375 0.268 0.034" />
       </geometry>
     </collision>
@@ -54,5 +55,5 @@
       <origin xyz="${-wheel_xpos-0.169} 0.169 ${-wheel_r+0.106}" rpy="0 0 0" />
       <geometry>
-        <box size="0.1 0.07 0.07"/>
+        <box size="0.1 0.07 0.07" />
       </geometry>
     </collision>
@@ -60,8 +61,8 @@
       <origin xyz="${-wheel_xpos-0.169} -0.169 ${-wheel_r+0.106}" rpy="0 0 0" />
       <geometry>
-        <box size="0.1 0.07 0.07"/>
-      </geometry>
-    </collision>
-    <xacro:box_inertial_with_origin  x="0.398" y="0.221" z="0.150" mass="10.0">
+        <box size="0.1 0.07 0.07" />
+      </geometry>
+    </collision>
+    <xacro:box_inertial_with_origin x="0.398" y="0.221" z="0.150" mass="10.0">
       <origin xyz="-0.15 0 0.03" rpy="0 0 0" />
     </xacro:box_inertial_with_origin>
@@ -78,5 +79,5 @@
         <origin xyz="0.115 0 0.635" rpy="0 0.56 0" />
         <geometry>
-          <box size="0.04 0.23 0.15"/>
+          <box size="0.04 0.23 0.15" />
         </geometry>
       </collision>
@@ -85,5 +86,5 @@
         <origin xyz="0.08 0 0.37" rpy="0 0 0" />
         <geometry>
-          <box size="0.06 0.24 0.40"/>
+          <box size="0.06 0.24 0.40" />
         </geometry>
       </collision>
@@ -92,5 +93,5 @@
         <origin xyz="-0.1 0 0.18" rpy="0 0 0" />
         <geometry>
-          <box size="0.42 0.24 0.03"/>
+          <box size="0.42 0.24 0.03" />
         </geometry>
       </collision>
@@ -99,5 +100,5 @@
         <origin xyz="-0.18 0 0.2" rpy="0 0 0" />
         <geometry>
-          <box size="0.35 0.408 0.005"/>
+          <box size="0.35 0.408 0.005" />
         </geometry>
       </collision>
@@ -106,5 +107,5 @@
         <origin xyz="-0.1 0 0.53" rpy="0 0 0" />
         <geometry>
-          <box size="0.32 0.42 0.02"/>
+          <box size="0.32 0.42 0.02" />
         </geometry>
       </collision>
@@ -122,5 +123,5 @@
         <origin xyz="-0.175 0 0.07" rpy="0 0.0 0" />
         <geometry>
-          <box size="0.3 0.33 0.2"/>
+          <box size="0.3 0.33 0.2" />
         </geometry>
       </collision>
@@ -128,9 +129,9 @@
   </link>
   <!-- Fixed offset from the floor to the center of the wheels -->
-  <link name="base_footprint"/>
+  <link name="base_footprint" />
   <joint name="base_footprint_joint" type="fixed">
-    <parent link="base_footprint"/>
-    <child link="base_link"/>
-    <origin xyz="0 0 ${wheel_r}" rpy="0 0 0"/>
+    <parent link="base_footprint" />
+    <child link="base_link" />
+    <origin xyz="0 0 ${wheel_r}" rpy="0 0 0" />
   </joint>
   <!-- Macro for defining wheels -->
@@ -146,5 +147,5 @@
         <origin xyz="0 0 0" rpy="0 ${pi/2} 0" />
         <geometry>
-          <cylinder radius="${wheel_r}" length="0.05"/>
+          <cylinder radius="${wheel_r}" length="0.05" />
         </geometry>
       </collision>
@@ -152,5 +153,5 @@
         <origin xyz="${0.033*reflect} 0 0" rpy="0 ${pi/2} 0" />
         <geometry>
-          <cylinder radius="0.064" length="0.016"/>
+          <cylinder radius="0.064" length="0.016" />
         </geometry>
       </collision>
@@ -161,11 +162,11 @@
     <joint name="${prefix}_wheel_joint" type="continuous">
       <axis xyz="1 0 0" rpy="0 0 0" />
-      <parent link="base_link"/>
-      <child link="${prefix}_wheel"/>
-      <origin xyz="0 ${0.163*reflect} 0" rpy="0 0 ${pi/2}"/>
+      <parent link="base_link" />
+      <child link="${prefix}_wheel" />
+      <origin xyz="0 ${0.163*reflect} 0" rpy="0 0 ${pi/2}" />
     </joint>
   </xacro:macro>
-  <xacro:wheel prefix="left" reflect="1"/>
-  <xacro:wheel prefix="right" reflect="-1"/>
+  <xacro:wheel prefix="left" reflect="1" />
+  <xacro:wheel prefix="right" reflect="-1" />
   <!-- Macro for defining caster wheels -->
   <xacro:macro name="caster_wheel" params="prefix reflect">
@@ -174,42 +175,45 @@
         <origin xyz="${-wheel_xpos-0.19} ${reflect*0.169} ${-wheel_r+0.04}" rpy="0 0 0" />
         <geometry>
-          <sphere radius="0.04"/>
+          <sphere radius="0.04" />
         </geometry>
       </collision>
     </link>
     <joint name="${prefix}_caster_wheel_joint" type="fixed">
-      <parent link="base_link"/>
-      <child link="${prefix}_caster_wheel"/>
+      <parent link="base_link" />
+      <child link="${prefix}_caster_wheel" />
     </joint>
   </xacro:macro>
-  <xacro:caster_wheel prefix="left" reflect="1"/>
-  <xacro:caster_wheel prefix="right" reflect="-1"/>
+  <xacro:caster_wheel prefix="left" reflect="1" />
+  <xacro:caster_wheel prefix="right" reflect="-1" />
   <!-- Define all sonars, if sonars_installed set to 1 -->
   <xacro:if value="${sonars_installed}">
     <xacro:sonar_hc-sr04 name="sonar_0" connected_to="base_link">
-      <origin xyz="0.01 -0.14 0.15" rpy="0 0 ${-pi/2}"/>
+      <origin xyz="0.01 -0.14 0.15" rpy="0 0 ${-pi/2}" />
     </xacro:sonar_hc-sr04>
     <xacro:sonar_hc-sr04 name="sonar_1" connected_to="base_link">
-      <origin xyz="0.08 -0.07 0.15" rpy="0 0 0.785"/>
+      <origin xyz="0.08 -0.07 0.15" rpy="0 0 0.785" />
     </xacro:sonar_hc-sr04>
     <xacro:sonar_hc-sr04 name="sonar_2" connected_to="base_link">
-      <origin xyz="0.08 -0.01 0.15" rpy="0 0 -0.785"/>
+      <origin xyz="0.08 -0.01 0.15" rpy="0 0 -0.785" />
     </xacro:sonar_hc-sr04>
     <xacro:sonar_hc-sr04 name="sonar_3" connected_to="base_link">
-      <origin xyz="0.08 0.04 0.15" rpy="0 0 0"/>
+      <origin xyz="0.08 0.04 0.15" rpy="0 0 0" />
     </xacro:sonar_hc-sr04>
     <xacro:sonar_hc-sr04 name="sonar_4" connected_to="base_link">
-      <origin xyz="0.01 0.14 0.15" rpy="0 0 ${pi/2}"/>
+      <origin xyz="0.01 0.14 0.15" rpy="0 0 ${pi/2}" />
     </xacro:sonar_hc-sr04>
   </xacro:if>
   <!-- Define camera -->
   <xacro:if value="${camera_extrinsics_file != ''}">
-    <xacro:property name="cam_extrinsics" value="${load_yaml(camera_extrinsics_file)}"/>
+    <xacro:property name="cam_extrinsics" value="${load_yaml(camera_extrinsics_file)}" />
     <xacro:raspi_camera name="raspicam" connected_to="base_link">
       <origin xyz="${cam_extrinsics['x']} ${cam_extrinsics['y']} ${cam_extrinsics['z']}"
-        rpy="${cam_extrinsics['roll']} ${cam_extrinsics['pitch']} ${cam_extrinsics['yaw']}"/>
+        rpy="${cam_extrinsics['roll']} ${cam_extrinsics['pitch']} ${cam_extrinsics['yaw']}" />
     </xacro:raspi_camera>
   </xacro:if>
-  <!-- Define Lidar -->
+  <xacro:teste connected_to="base_link">
+    <origin xyz="-0.15 0 0.16" rpy="0 0 ${-pi/2}" />
+  </xacro:teste>
+  <!-- Define Lidar
   <xacro:if value="${lidar_extrinsics_file != ''}">
     <xacro:property name="lidar_extrinsics" value="${load_yaml(lidar_extrinsics_file)}"/>
@@ -219,3 +223,5 @@
     </xacro:ur50_lidar>
   </xacro:if>
+  -->
+  <xacro:include filename="model.sdf" />
 </robot>
