Commit message: update marker

File: magni_description/urdf/model.urdf (robot description, URDF)
Before this commit: robot magni_base, 2 links, 1 joints
Links:
- link link_0: geometry collision mesh filename=base.dae scale=0.2 0.5 1; visual mesh filename=base.dae scale=0.2 0.5 1
- link marker_pad: geometry collision box size=0.1 0.12 1e-5; visual box size=0.1 0.12 1e-5
